Commit message: calibration

File: urdf/ur3_robotiq_unit.urdf.xacro (robot description, xacro)
@@ -51,4 +51,5 @@
 		gripper_name:='gripper' gripper_use_fake_hardware:='true'
 		gripper_fake_sensor_commands:='false' gripper_com_port:='/tmp/ttyUR'
+		use_calib_probe:='false'
 	">
 		<xacro:ur_robot
@@ -79,5 +80,4 @@
 			output_recipe_filename="${output_recipe_filename}"
 			input_recipe_filename="${input_recipe_filename}"
-			reverse_ip="0.0.0.0"
 			reverse_port="${reverse_port}"
 			script_sender_port="${script_sender_port}"
@@ -116,4 +116,18 @@
 			fake_sensor_commands="${gripper_fake_sensor_commands}"
 			com_port="${gripper_com_port}"/>
+		<xacro:if value="${use_calib_probe}">
+			<link name="${tf_prefix}probe_link">
+				<visual>
+					<geometry>
+						<mesh filename="package://ur_robotiq/meshes/triangle.obj"/>
+					</geometry>
+				</visual>
+			</link>
+			<joint name="${tf_prefix}probe_joint" type="fixed">
+				<parent link="${tf_prefix}tool0"/>
+				<child link="${tf_prefix}probe_link"/>
+				<origin xyz="0 0 0.15" rpy="1.57 0 0"/>
+			</joint>
+		</xacro:if>
 	</xacro:macro>
 	<xacro:if value="$(arg instantiate_unit)">

Commit message: missing calibration

File: urdf/ur3_robotiq_unit.urdf.xacro (robot description, xacro)
@@ -2,5 +2,5 @@
 <robot xmlns:xacro="http://wiki.ros.org/xacro" name="ur3_robotiq_unit">
 	<xacro:include filename="$(find ur_description)/urdf/ur_macro.xacro"/>
-	<xacro:include filename="$(find ur_robot_driver)/urdf/ur.ros2_control.xacro"/>
+	<xacro:include filename="$(find ur_description)/urdf/ur.ros2_control.xacro"/>
 	<xacro:include filename="$(find robotiq_description)/urdf/ur_to_robotiq_adapter.urdf.xacro"/>
 	<xacro:include filename="$(find robotiq_description)/urdf/robotiq_2f_85_macro.urdf.xacro"/>
@@ -64,14 +64,7 @@
 			safety_pos_margin="0.15"
 			safety_k_position="20"
-			force_abs_paths="false">
-			<origin xyz="${base_xyz}" rpy="${base_rpy}"/>
-		</xacro:ur_robot>
-		<xacro:ur_ros2_control
-			name="${arm_name}"
-			tf_prefix="${tf_prefix}"
-			kinematics_parameters_file="${kinematics_parameters_file}"
-			transmission_hw_interface="hardware_interface/PositionJointInterface"
-			use_mock_hardware="${use_mock_hardware}"
-			mock_sensor_commands="${mock_sensor_commands}"
+			generate_ros2_control_tag="true"
+			use_fake_hardware="${use_mock_hardware}"
+			fake_sensor_commands="${mock_sensor_commands}"
 			headless_mode="${headless_mode}"
 			initial_positions="${initial_positions}"
@@ -92,5 +85,7 @@
 			tool_tx_idle_chars="${tool_tx_idle_chars}"
 			tool_device_name="${tool_device_name}"
-			tool_tcp_port="${tool_tcp_port}"/>
+			tool_tcp_port="${tool_tcp_port}">
+			<origin xyz="${base_xyz}" rpy="${base_rpy}"/>
+		</xacro:ur_robot>
 		<xacro:ur_to_robotiq
 			prefix="${tf_prefix}"

Commit message: min grasp force

File: urdf/ur3_robotiq_unit.urdf.xacro (robot description, xacro)
@@ -6,7 +6,8 @@
 	<xacro:include filename="$(find robotiq_description)/urdf/robotiq_2f_85_macro.urdf.xacro"/>
 	<xacro:arg name="instantiate_unit" default="false"/>
+	<xacro:arg name="gripper_closed_position" default="0.8"/>
 	<xacro:arg name="kinematics_parameters_file" default="$(find ur_description)/config/ur3/default_kinematics.yaml"/>
 	<xacro:property name="default_initial_positions" value="${xacro.load_yaml('$(find ur_description)/config/initial_positions.yaml')}"/>
-	<xacro:macro name="robotiq_minimal_ros2_control" params="name prefix use_fake_hardware fake_sensor_commands com_port">
+	<xacro:macro name="robotiq_minimal_ros2_control" params="name prefix use_fake_hardware fake_sensor_commands com_port gripper_closed_position">
 		<ros2_control name="${name}" type="system">
 			<hardware>
@@ -18,8 +19,8 @@
 				<xacro:unless value="${use_fake_hardware}">
 					<plugin>robotiq_driver/RobotiqGripperHardwareInterface</plugin>
-					<param name="gripper_closed_position">0.7929</param>
+					<param name="gripper_closed_position">${gripper_closed_position}</param>
 					<param name="COM_port">${com_port}</param>
-					<param name="gripper_speed_multiplier">1.0</param>
-					<param name="gripper_force_multiplier">0.5</param>
+					<param name="gripper_speed_multiplier">0.01</param>
+					<param name="gripper_force_multiplier">0.01</param>
 				</xacro:unless>
 			</hardware>
@@ -51,5 +52,5 @@
 		tool_device_name:='/tmp/ttyUR' tool_tcp_port:='54321'
 		gripper_name:='gripper' gripper_use_fake_hardware:='true'
-		gripper_fake_sensor_commands:='false' gripper_com_port:='/tmp/ttyUR'
+		gripper_fake_sensor_commands:='false' gripper_com_port:='/tmp/ttyUR' gripper_closed_position:='0.8'
 		use_calib_probe:='false'
 	">
@@ -111,5 +112,6 @@
 			use_fake_hardware="${gripper_use_fake_hardware}"
 			fake_sensor_commands="${gripper_fake_sensor_commands}"
-			com_port="${gripper_com_port}"/>
+			com_port="${gripper_com_port}"
+			gripper_closed_position="${gripper_closed_position}"/>
 		<xacro:if value="${use_calib_probe}">
 			<link name="${tf_prefix}probe_link">

Commit message: wip gello ros

File: urdf/ur3_robotiq_unit.urdf.xacro (robot description, xacro)
@@ -7,7 +7,8 @@
 	<xacro:arg name="instantiate_unit" default="false"/>
 	<xacro:arg name="gripper_closed_position" default="0.82"/>
+	<xacro:arg name="gripper_force_multiplier" default="0.01"/>
 	<xacro:arg name="kinematics_parameters_file" default="$(find ur_description)/config/ur3/default_kinematics.yaml"/>
 	<xacro:property name="default_initial_positions" value="${xacro.load_yaml('$(find ur_description)/config/initial_positions.yaml')}"/>
-	<xacro:macro name="robotiq_minimal_ros2_control" params="name prefix use_fake_hardware fake_sensor_commands com_port gripper_closed_position">
+	<xacro:macro name="robotiq_minimal_ros2_control" params="name prefix use_fake_hardware fake_sensor_commands com_port gripper_closed_position gripper_force_multiplier">
 		<ros2_control name="${name}" type="system">
 			<hardware>
@@ -22,5 +23,5 @@
 					<param name="COM_port">${com_port}</param>
 					<param name="gripper_speed_multiplier">0.01</param>
-					<param name="gripper_force_multiplier">0.01</param>
+					<param name="gripper_force_multiplier">${gripper_force_multiplier}</param>
 				</xacro:unless>
 			</hardware>
@@ -52,5 +53,6 @@
 		tool_device_name:='/tmp/ttyUR' tool_tcp_port:='54321'
 		gripper_name:='gripper' gripper_use_fake_hardware:='true'
-		gripper_fake_sensor_commands:='false' gripper_com_port:='/tmp/ttyUR' gripper_closed_position:='0.8'
+		gripper_fake_sensor_commands:='false' gripper_com_port:='/tmp/ttyUR'
+		gripper_closed_position:='0.8' gripper_force_multiplier:='0.01'
 		use_calib_probe:='false'
 	">
@@ -114,5 +116,6 @@
 			fake_sensor_commands="${gripper_fake_sensor_commands}"
 			com_port="${gripper_com_port}"
-			gripper_closed_position="${gripper_closed_position}"/>
+			gripper_closed_position="${gripper_closed_position}"
+			gripper_force_multiplier="${gripper_force_multiplier}"/>
 		<xacro:if value="${use_calib_probe}">
 			<link name="${tf_prefix}probe_link">

Commit message: initial positions

File: urdf/ur3_robotiq_unit.urdf.xacro (robot description, xacro)
@@ -9,5 +9,6 @@
 	<xacro:arg name="gripper_force_multiplier" default="0.01"/>
 	<xacro:arg name="kinematics_parameters_file" default="$(find ur_description)/config/ur3/default_kinematics.yaml"/>
-	<xacro:property name="default_initial_positions" value="${xacro.load_yaml('$(find ur_description)/config/initial_positions.yaml')}"/>
+	<xacro:property name="default_initial_positions_file" value="$(find ur_robotiq)/config/initial_positions.yaml"/>
+	<xacro:property name="default_initial_positions" value="${xacro.load_yaml(default_initial_positions_file)['left']}"/>
 	<xacro:macro name="robotiq_minimal_ros2_control" params="name prefix use_fake_hardware fake_sensor_commands com_port gripper_closed_position gripper_force_multiplier">
 		<ros2_control name="${name}" type="system">

Commit message: gripper initial positions

File: urdf/ur3_robotiq_unit.urdf.xacro (robot description, xacro)
@@ -11,5 +11,5 @@
 	<xacro:property name="default_initial_positions_file" value="$(find ur_robotiq)/config/initial_positions.yaml"/>
 	<xacro:property name="default_initial_positions" value="${xacro.load_yaml(default_initial_positions_file)['left']}"/>
-	<xacro:macro name="robotiq_minimal_ros2_control" params="name prefix use_fake_hardware fake_sensor_commands com_port gripper_closed_position gripper_force_multiplier">
+	<xacro:macro name="robotiq_minimal_ros2_control" params="name prefix use_fake_hardware initial_positions fake_sensor_commands com_port gripper_closed_position gripper_force_multiplier">
 		<ros2_control name="${name}" type="system">
 			<hardware>
@@ -30,5 +30,5 @@
 				<command_interface name="position"/>
 				<state_interface name="position">
-					<param name="initial_value">0.7929</param>
+					<param name="initial_value">${initial_positions['gripper_joint']}</param>
 				</state_interface>
 				<state_interface name="velocity"/>
@@ -115,4 +115,5 @@
 			prefix="${tf_prefix}"
 			use_fake_hardware="${gripper_use_fake_hardware}"
+			initial_positions="${initial_positions}"
 			fake_sensor_commands="${gripper_fake_sensor_commands}"
 			com_port="${gripper_com_port}"
