Commit message: ur mia control

File: urdf/ur_mia_unit.urdf.xacro (robot description, xacro)
@@ -1,4 +1,4 @@
 <?xml version="1.0"?>
-<robot xmlns:xacro="http://wiki.ros.org/xacro" name="ur5_mia_unit">
+<robot xmlns:xacro="http://wiki.ros.org/xacro" name="ur_mia_unit">
 	<xacro:include filename="$(find ur_description)/urdf/ur_macro.xacro"/>
 	<xacro:include filename="$(find ur_description)/urdf/ur.ros2_control.xacro"/>
@@ -10,5 +10,5 @@
 	<xacro:property name="default_initial_positions_file" value="$(find ur_robotiq)/config/initial_positions.yaml"/>
 	<xacro:property name="default_initial_positions" value="${xacro.load_yaml(default_initial_positions_file)['left']}"/>
-	<xacro:macro name="ur5_mia_unit" params="
+	<xacro:macro name="ur_mia_unit" params="
 		arm_name:='ur5' tf_prefix:='' parent:='world' base_xyz:='0 0 0' base_rpy:='0 0 0'
 		laterality:='right'
@@ -111,5 +111,5 @@
 		<xacro:property name="instantiate_initial_positions_all" value="${xacro.load_yaml(default_initial_positions_file)}"/>
 		<xacro:if value="${'right' == '$(arg laterality)'}">
-			<xacro:ur5_mia_unit
+			<xacro:ur_mia_unit
 				laterality="$(arg laterality)"
 				initial_positions="${instantiate_initial_positions_all['right']}"
@@ -117,5 +117,5 @@
 		</xacro:if>
 		<xacro:if value="${'left' == '$(arg laterality)'}">
-			<xacro:ur5_mia_unit
+			<xacro:ur_mia_unit
 				laterality="$(arg laterality)"
 				initial_positions="${instantiate_initial_positions_all['left']}"

File: urdf/ur_robotiq_unit.urdf.xacro (robot description, xacro)
@@ -1,4 +1,4 @@
 <?xml version="1.0"?>
-<robot xmlns:xacro="http://wiki.ros.org/xacro" name="ur3e_robotiq_unit">
+<robot xmlns:xacro="http://wiki.ros.org/xacro" name="ur_robotiq_unit">
 	<xacro:include filename="$(find ur_description)/urdf/ur_macro.xacro"/>
 	<xacro:include filename="$(find ur_description)/urdf/ur.ros2_control.xacro"/>
@@ -30,5 +30,5 @@
 				<command_interface name="position"/>
 				<state_interface name="position">
-					<param name="initial_value">${initial_positions['gripper_joint']}</param>
+					<param name="initial_value">${initial_positions['gripper_joint'] if 'gripper_joint' in initial_positions else 0.0}</param>
 				</state_interface>
 				<state_interface name="velocity"/>
@@ -40,5 +40,5 @@
 		</ros2_control>
 	</xacro:macro>
-	<xacro:macro name="ur3e_robotiq_unit" params="
+	<xacro:macro name="ur_robotiq_unit" params="
 		arm_name:='ur3e' tf_prefix:='' parent:='world' base_xyz:='0 0 0' base_rpy:='0 0 0'
 		use_mock_hardware:='true' mock_sensor_commands:='false' headless_mode:='false'
@@ -137,5 +137,5 @@
 	<xacro:if value="$(arg instantiate_unit)">
 		<link name="world"/>
-		<xacro:ur3e_robotiq_unit
+		<xacro:ur_robotiq_unit
 			kinematics_parameters_file="$(arg kinematics_parameters_file)"/>
 	</xacro:if>
